Commit message: fix pid

File: my_robot/description/camera.xacro (robot description, xacro)
@@ -4,5 +4,5 @@
   <xacro:include filename="$(find my_robot)/description/_d435i.urdf.xacro"/>
   <xacro:sensor_d435i parent="chassis_link" use_nominal_extrinsics="$(arg use_nominal_extrinsics)">
-    <origin xyz="0.25 0 0.12" rpy="0 0 0"/>
+    <origin xyz="0.243 0 0.085" rpy="0 0 0"/>
   </xacro:sensor_d435i>
 </robot>

File: my_robot/description/ros2_control.xacro (robot description, xacro)
@@ -7,14 +7,18 @@
                 <param name="left_wheel_name">left_wheel_joint</param>
                 <param name="right_wheel_name">right_wheel_joint</param>
-                <param name="loop_rate">100</param>
+                <param name="loop_rate">40</param>
                 <param name="device">/dev/ttyUSB0</param>
-                <param name="baud_rate">57600</param>
+                <param name="baud_rate">115200</param>
                 <param name="timeout_ms">1000</param>
-                <param name="enc_counts_per_rev_r">1560</param>
-                <param name="enc_counts_per_rev_l">1560</param>
-                <param name="pid_p">20</param>
-                <param name="pid_d">12</param>
-                <param name="pid_i">0</param>
-                <param name="pid_o">50</param>
+                <param name="enc_counts_per_rev_r">39300</param>
+                <param name="enc_counts_per_rev_l">39300</param>
+                <param name="pid_p_r">21</param>
+                <param name="pid_d_r">15</param>
+                <param name="pid_i_r">0</param>
+                <param name="pid_o_r">1000</param>
+                <param name="pid_p_l">20</param>
+                <param name="pid_d_l">10</param>
+                <param name="pid_i_l">0</param>
+                <param name="pid_o_l">1000</param>
             </hardware>
             <joint name="left_wheel_joint">
