Commit message: 2-2

File: my_robot/description/lidar.xacro (robot description, xacro)
@@ -4,5 +4,5 @@
         <parent link="chassis_link"/>
         <child link="laser_frame"/>
-        <origin xyz="0.097 0 0.14" rpy="0 0 0"/>
+        <origin xyz="0.097 0 0.14" rpy="0 0 ${9.85*pi/10}"/>
     </joint>
     <link name="laser_frame">

Commit message: 21-3

File: my_robot/description/lidar.xacro (robot description, xacro)
@@ -4,5 +4,5 @@
         <parent link="chassis_link"/>
         <child link="laser_frame"/>
-        <origin xyz="0.097 0 0.14" rpy="0 0 ${9.85*pi/10}"/>
+        <origin xyz="0.097 0 0.14" rpy="0 0 0"/>
     </joint>
     <link name="laser_frame">

File: my_robot/description/robot.urdf.xacro (robot description, xacro)
@@ -2,5 +2,5 @@
 <robot xmlns:xacro="http://www.ros.org/wiki/xacro"  name="robot">
     <xacro:arg name="use_ros2_control" default="true"/>
-    <xacro:arg name="sim_mode" default="false"/>
+    <xacro:arg name="sim_mode" default="true"/>
     <xacro:include filename="robot_core.xacro"/>
     <xacro:if value="$(arg use_ros2_control)">
