Commit message: 11-3

File: my_robot/description/robot_core.xacro (robot description, xacro)
@@ -27,5 +27,5 @@
     <xacro:property name="chassis_height" value="0.06685"/>
     <xacro:property name="chassis_mass" value="3.0"/>
-    <xacro:property name="wheel_radius" value="0.033"/>
+    <xacro:property name="wheel_radius" value="0.0325"/>
     <xacro:property name="wheel_thickness" value="0.026"/>
     <xacro:property name="wheel_mass" value="0.05"/>

File: my_robot/description/ros2_control.xacro (robot description, xacro)
@@ -7,5 +7,5 @@
                 <param name="left_wheel_name">left_wheel_joint</param>
                 <param name="right_wheel_name">right_wheel_joint</param>
-                <param name="loop_rate">100</param>
+                <param name="loop_rate">50</param>
                 <param name="device">/dev/ttyUSB0</param>
                 <param name="baud_rate">57600</param>

Commit message: 2-4

File: my_robot/description/robot_core.xacro (robot description, xacro)
@@ -27,5 +27,5 @@
     <xacro:property name="chassis_height" value="0.06685"/>
     <xacro:property name="chassis_mass" value="3.0"/>
-    <xacro:property name="wheel_radius" value="0.0325"/>
+    <xacro:property name="wheel_radius" value="0.033"/>
     <xacro:property name="wheel_thickness" value="0.026"/>
     <xacro:property name="wheel_mass" value="0.05"/>
